File: Sensor Cluster Team/SensorPod ECAD/SensorPod.sch (EAGLE design)
At the start: 40 parts, among them J1 BMP388, J2 BMP388, J3 BMP388, J4 BMP388, J5 BMP388, J6 BMP388

Commit message: v0_0_1 Sensor Pod Finished
Parts:
- removed TP2, TP3, TP4, TP5, TP6: TPB1,27, testpad:TPB1,27
- added C13: 587-3766-1-ND, rcl:C-EUC0402
- added C14: 490-7998-1-ND, rcl:C-EUC0402
- added IC1: SST25PF040CT-40E_SN, SamacSys_Parts:SST25PF040CT-40E_SN
- added TP21: TPB1,27, testpad:TPB1,27
Connections:
- removed net N$1: J1.INT, TP1.TP
- removed net N$2: J2.INT, TP2.TP
- removed net N$3: J3.INT, TP3.TP
- removed net N$4: J4.INT, TP4.TP
- removed net N$5: J5.INT, TP5.TP
- removed net N$6: J6.INT, TP6.TP
- new net C1_INT: J1.INT, J8.7, TP1.TP
- new net CS_MEM: IC1.CE#, J8.8, TP21.TP
- net CS_1_BAK: now also J8.5; no longer J8.4
- net CS_1_MAIN: now also J8.6; no longer J7.4
- net CS_2_MAIN: now also J8.4; no longer J7.3
- net CS_3_BAK: now also J8.1; no longer J8.2
- net CS_3_MAIN: now also J8.2; no longer J7.2
- net GND: now also C13.2, C14.2, IC1.VSS; no longer J8.1
- net MISO_BAK: now also J7.2; no longer J8.6
- net MISO_MAIN: now also IC1.SO/SIO1, J7.5; no longer J7.6
- net MOSI_BAK: now also J7.3; no longer J8.7
- net MOSI_MAIN: now also IC1.SI/SIO0, J7.6; no longer J7.7
- net SCK_BAK: now also J7.4; no longer J8.5
- net SCK_MAIN: now also IC1.SCK, J7.7; no longer J7.5
- net VCC: now also C13.1, C14.1, IC1.HOLD#, IC1.VDD, IC1.WP#; no longer J8.8
Other:
- note added: "EEPROM"
- note added: "Notes: 1. 490-7998-1-ND is an AEC-Q200 qualified 100nF capacitor. 2. INT pins are DNC. Broke out one of them just in case we want to experiment."
- note added: "Notes: 1. 587-3766-1-ND is an AEC-Q200 qualified 1uF capacitor."
- note removed: "Notes: 1. 490-7998-1-ND is an AEC-Q200 qualified 100nF capacitor. 2. INT pins are DNC, routed to test points in case we decide to use them later."
